File: Electronics/_restore_backup_2026-08-22T19-55-00-620/Hexapod PCB 2.kicad_sch (KiCad schematic)
At the start: 69 parts, among them J1 XT60, J2 leg1, J3 leg2, J4 leg3, J5 leg4, J6 leg5, J7 leg6, J8 USB_C_Receptacle_USB2.0_16P, Q1 IRF4905, Q2 Q_NPN_BCE, Q3 Q_NPN_BCE, SW1 SW_SPST, SW2 SW_SPST, SW3 SW_SPST, U1 TPS563201, U2 TPS563201, U3 ESP32-S3-WROOM-1, U4 USBLC6-2P6, U5 BNO055, U6 INA226

Commit message: finished the schmeatics by redesigning the INA226 , set all of the footprint for the schematics
Parts:
- J2, J3, J4, J5, J6, J7: footprint Connector_JST:JST_PH_B3B-PH-K_1x03_P2.00mm_Vertical -> (none)
Changed lines of the file:
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@@
 			)
 		)
-		(property "Footprint" "Connector_JST:JST_PH_B3B-PH-K_1x03_P2.00mm_Vertical"
+		(property "Footprint" ""
 			(at 247.65 39.37 0)
 			(hide yes)
@@
 			)
 		)
-		(property "Footprint" "Connector_JST:JST_PH_B3B-PH-K_1x03_P2.00mm_Vertical"
+		(property "Footprint" ""
 			(at 278.13 39.37 0)
 			(hide yes)
@@
 			)
 		)
-		(property "Footprint" "Connector_JST:JST_PH_B3B-PH-K_1x03_P2.00mm_Vertical"
+		(property "Footprint" ""
 			(at 278.13 30.48 0)
 			(hide yes)
@@
 			)
 		)
-		(property "Footprint" "Connector_JST:JST_PH_B3B-PH-K_1x03_P2.00mm_Vertical"
+		(property "Footprint" ""
 			(at 247.65 30.48 0)
 			(hide yes)
@@
 			)
 		)
-		(property "Footprint" "Connector_JST:JST_PH_B3B-PH-K_1x03_P2.00mm_Vertical"
+		(property "Footprint" ""
 			(at 278.13 21.59 0)
 			(hide yes)
@@
 			)
 		)
-		(property "Footprint" "Connector_JST:JST_PH_B3B-PH-K_1x03_P2.00mm_Vertical"
+		(property "Footprint" ""
 			(at 247.65 21.59 0)
 			(hide yes)
