File: Electronics/KiCAD project/Hexapod PCB 2.kicad_pcb (KiCad board)
At the start: 4 copper layers, 53 x 85 mm, 80 parts, among them J1 XT60, J2 leg1, J3 leg2, J4 leg3, J5 leg4, J6 leg5, J7 leg6, J8 USB_C_Receptacle_USB2.0_16P, Q1 IRF4905, Q2 Q_NPN_BCE, Q3 Q_NPN_BCE, SW2 SW_SPST, SW3 SW_SPST, U1 TPS563201, U2 TPS563201, U3 ESP32-S3-WROOM-1, U4 USBLC6-2P6, U5 BNO055, U6 INA226

Commit message: added CAD files added Renders changed the PCB connector footprints added PCB BOM added Hexapod BOM made the project  file structure
Parts:
- removed G***: LOGO, LOGO
- J2, J3, J4, J5, J6, J7: footprint Connector_JST:JST_PH_B3B-PH-K_1x03_P2.00mm_Vertical -> Connector_JST:JST_XH_B3B-XH-A_1x03_P2.50mm_Vertical
- moved J3 7.73 mm to (139.9, 91.3), turned to 90 degrees
- moved J2 5.11 mm to (132.6, 91.3), turned to 90 degrees
- moved J5 2.74 mm to (174.0, 84.0)
- moved J6 1.87 mm to (174.0, 91.0)
- moved J7 1.61 mm to (174.0, 98.0)
- moved J4 0.64 mm to (132.7, 97.4)
Routing:
- net BUS1: track 81.4 -> 68.8 mm
- net BUS2: track 54.1 -> 55.0 mm
Other:
- board text removed: "67"
- board text removed: "MadHex"
- board text removed: "pcbway"
