File: Electronics/KiCAD project/Hexapod PCB 2.kicad_sch (KiCad schematic)
At the start: 79 parts, among them J1 XT60, J2 leg1, J3 leg2, J4 leg3, J5 leg4, J6 leg5, J7 leg6, J8 USB_C_Receptacle_USB2.0_16P, Q1 IRF4905, Q2 Q_NPN_BCE, Q3 Q_NPN_BCE, SW2 SW_SPST, SW3 SW_SPST, U1 TPS563201, U2 TPS563201, U3 ESP32-S3-WROOM-1, U4 USBLC6-2P6, U5 BNO055, U6 INA226

Commit message: added CAD files added Renders changed the PCB connector footprints added PCB BOM added Hexapod BOM made the project  file structure
Parts:
- J1: footprint Connector_AMASS:AMASS_XT60PW-M_1x02_P7.20mm_Horizontal -> Connector_AMASS:AMASS_XT60-M_1x02_P7.20mm_Vertical
- J2, J3, J4, J5, J6, J7: footprint Connector_JST:JST_PH_B3B-PH-K_1x03_P2.00mm_Vertical -> Connector_JST:JST_XH_B3B-XH-A_1x03_P2.50mm_Vertical
Changed lines of the file:
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@@
 			)
 		)
-		(property "Footprint" "Connector_JST:JST_PH_B3B-PH-K_1x03_P2.00mm_Vertical"
+		(property "Footprint" "Connector_JST:JST_XH_B3B-XH-A_1x03_P2.50mm_Vertical"
 			(at 248.92 44.45 0)
 			(hide yes)
@@
 			)
 		)
-		(property "Footprint" "Connector_JST:JST_PH_B3B-PH-K_1x03_P2.00mm_Vertical"
+		(property "Footprint" "Connector_JST:JST_XH_B3B-XH-A_1x03_P2.50mm_Vertical"
 			(at 279.4 44.45 0)
 			(hide yes)
@@
 			)
 		)
-		(property "Footprint" "Connector_AMASS:AMASS_XT60PW-M_1x02_P7.20mm_Horizontal"
+		(property "Footprint" "Connector_AMASS:AMASS_XT60-M_1x02_P7.20mm_Vertical"
 			(at 20.32 27.94 0)
 			(hide yes)
@@
 			)
 		)
-		(property "Footprint" "Connector_JST:JST_PH_B3B-PH-K_1x03_P2.00mm_Vertical"
+		(property "Footprint" "Connector_JST:JST_XH_B3B-XH-A_1x03_P2.50mm_Vertical"
 			(at 279.4 35.56 0)
 			(hide yes)
@@
 			)
 		)
-		(property "Footprint" "Connector_JST:JST_PH_B3B-PH-K_1x03_P2.00mm_Vertical"
+		(property "Footprint" "Connector_JST:JST_XH_B3B-XH-A_1x03_P2.50mm_Vertical"
 			(at 248.92 35.56 0)
 			(hide yes)
@@
 			)
 		)
-		(property "Footprint" "Connector_JST:JST_PH_B3B-PH-K_1x03_P2.00mm_Vertical"
+		(property "Footprint" "Connector_JST:JST_XH_B3B-XH-A_1x03_P2.50mm_Vertical"
 			(at 279.4 26.67 0)
 			(hide yes)
@@
 			)
 		)
-		(property "Footprint" "Connector_JST:JST_PH_B3B-PH-K_1x03_P2.00mm_Vertical"
+		(property "Footprint" "Connector_JST:JST_XH_B3B-XH-A_1x03_P2.50mm_Vertical"
 			(at 248.92 26.67 0)
 			(hide yes)

Commit message: added PWRflags into the scmatics and solved some ERC problems
Connections:
- no-connect marks 7 -> 30

Commit message: update PCB, BOM, README, add firmware
Parts:
- removed Q1: IRF4905, Package_TO_SOT_SMD:TO-263-2, symbol Transistor_FET:IRF4905
- removed Q2, Q3: Q_NPN_BCE, Package_TO_SOT_SMD:SOT-23, symbol Transistor_BJT:Q_NPN_BCE
- removed R27: RS, Resistor_SMD:R_2512_6332Metric, symbol Device:R
- added C26: 0.1uF, Capacitor_SMD:C_0805_2012Metric, symbol Device:C
- added D3, D4: SS34, Diode_SMD:D_SMA, symbol Diode:SS34
- added D5: BZT52C12, Diode_SMD:D_SOD-123, symbol Device:D_Zener
- added Q1: NTMFS5C404NLT1G, n-mosfet:NTMFS4C022N, symbol NTMFS5C404NLT1G:NTMFS5C404NLT1G
- added Q2, Q3: MMBT3904, Package_TO_SOT_SMD:SOT-23, symbol Transistor_BJT:MMBT3904
- added R28: 100k, Resistor_SMD:R_0805_2012Metric, symbol Device:R
- added R29: 1k, Resistor_SMD:R_0805_2012Metric, symbol Device:R
- D1: value D_TVS -> SMBJ10CA
- R1: value 100k -> 10k
- R2: value 54.9k -> 59k
- R23: value 10k -> 2m; footprint Resistor_SMD:R_0805_2012Metric -> Resistor_SMD:R_2512_6332Metric
- R24: value 10k -> 1k
- R8: value 51k -> 100k
Connections:
- net +3.3V: no longer R23.1, R24.1
- net +5V: now also R5.1, D3.1 (K), D4.1 (K); no longer C7.2, C8.2, J8.A4 (VBUS), J8.A9 (VBUS), J8.B4 (VBUS), J8.B9 (VBUS), L1.2, R2.2, U4.5 (VBUS)
- net +BATT: now also D1.1 (A1), R1.2, R23.1, U6.10 (Vin+)
- net BUS1: now also R24.2, Q2.3 (C); no longer U3.36 (RXD0)
- net BUS2: now also Q3.3 (C), R29.2; no longer U3.11 (IO18)
- net GND: now also D1.2 (A2), C26.2, D5.2 (A), Q1.1 (S_1), Q1.2 (S_2), Q1.3 (S_3), Q2.2 (E), Q3.2 (E), R28.2; no longer D1.1 (A1), J1.1 (Pin_1), R1.1
- net SERVO-POWER: now also R23.2, R4.1; no longer D1.2 (A2), U6.10 (Vin+)
- net TX1: now also U3.4 (IO4); no longer U3.37 (TXD0)
- net VBATT-SENSE: now also C26.1
- net at R22.1, U6.2 (A0): no longer R24.2
- net at R20.1, U6.1 (A1): no longer R23.2
- net at U3.5 (IO5): now also R24.1
- net at R10.2: now also Q2.1 (B)
- net at R12.2: now also Q3.1 (B)
- removed net EN: R4.1, R5.1
- new net: R29.1, U3.11 (IO18)
- new net: D5.1 (K), Q1.4 (G), R1.1, R28.1
- new net: D3.2 (A), J8.A4 (VBUS), J8.A9 (VBUS), J8.B4 (VBUS), J8.B9 (VBUS), U4.5 (VBUS)
- new net -BATT: J1.1 (Pin_1), Q1.5 (D_1), Q1.6 (D_2), Q1.7 (D_3), Q1.8 (D_4), Q1.9 (D_5)
- new net 5v_buck: C7.2, C8.2, D4.2 (A), L1.2, R2.2
Other:
- note added: "filtering stage"
- moved on the sheet: C1, C2, C20, C21, C22, C23, C24, C25, D1, D2, J1, J2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
